File: dlock13.sch (EAGLE design)
At the start: 18 parts, among them IC2 7805T, Q1 IRLZ44Z, Q2 IRLZ44Z

Commit message: Updated.
Parts:
- removed R12: 4.7k, rcl:R-EU_0207/10
- R5: value 470 -> 4.7k
Connections:
- removed net N$6: Q2.S, R12.2
- net GND: now also Q2.S; no longer R12.1
Changed lines of the file:
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@@
 <part name="GND4" library="supply1" deviceset="GND" device=""/>
 <part name="Q2" library="transistor-power" deviceset="IRLZ44Z" device=""/>
-<part name="R5" library="resistor" deviceset="R-EU_" device="0204/7" value="470"/>
-<part name="R12" library="rcl" deviceset="R-EU_" device="0207/10" value="4.7k"/>
+<part name="R5" library="resistor" deviceset="R-EU_" device="0204/7" value="4.7k"/>
 <part name="GND2" library="supply1" deviceset="GND" device=""/>
 <part name="P+3" library="supply1" deviceset="VCC" device=""/>
@@
 <instance part="Q2" gate="G$1" x="68.58" y="50.8"/>
 <instance part="R5" gate="G$1" x="55.88" y="48.26"/>
-<instance part="R12" gate="G$1" x="71.12" y="38.1" rot="R90"/>
 <instance part="GND2" gate="1" x="71.12" y="27.94"/>
 <instance part="P+3" gate="VCC" x="99.06" y="25.4"/>
@@
 <segment>
 <pinref part="GND2" gate="1" pin="GND"/>
-<pinref part="R12" gate="G$1" pin="1"/>
-<wire x1="71.12" y1="30.48" x2="71.12" y2="33.02" width="0.1524" layer="91"/>
+<pinref part="Q2" gate="G$1" pin="S"/>
+<wire x1="71.12" y1="30.48" x2="71.12" y2="45.72" width="0.1524" layer="91"/>
 </segment>
 <segment>
@@
 </segment>
 </net>
-<net name="N$6" class="0">
-<segment>
-<pinref part="R12" gate="G$1" pin="2"/>
-<pinref part="Q2" gate="G$1" pin="S"/>
-<wire x1="71.12" y1="43.18" x2="71.12" y2="45.72" width="0.1524" layer="91"/>
-</segment>
-</net>

Commit message: Add vidarkr's changes. Produced and In use.
Parts:
- removed SV1: (no value), con-ml:ML26
- added C3: (no value), rcl:CPOL-EUE1,8-4LARGEPADS
- added D1: 1N4004DO41-10LARGEPADS, diode:1N4004DO41-10LARGEPADS
- added PICONNECTOR: RASPBERRY-PI, RaspberryPi:RASPBERRY-PI_REV1PIWITHPADSREMOVED
- C1, C2: device capacitor-wima:C2,5-3 -> capacitor-wima:CC2.5-3LARGEPADS
- D4: value 1N4004 -> 1N4004DO41-10LARGEPADS; device diode:1N4004 -> diode:1N4004DO41-10LARGEPADS
- J3: device con-jack:DCJ0303 -> con-jack:DCJ0303DCJ0303LARGEPADS
- JP2: device pinhead:PINHD-1X2 -> pinhead:PINHD-1X21X02LARGEPADS
- LED1: device led:LED5MM -> led:LEDLED5MMLARGEPADS
- R1, R2, R3: device rcl:R-EU_0207/10 -> rcl:R-EU_0207/10LARGEPADS
- R10, R5: device resistor:R-EU_0204/7 -> rcl:R-EU_0207/10LARGEPADS
- SV2: device con-lstb:MA04-1 -> con-lstb:MA04-1MA04-1LARGEPADS
Connections:
- removed net N$1: R5.1, SV1.22
- removed net N$12: JP2.1, SV1.15
- removed net N$8: JP1.1, R1.1, SV1.16
- removed net N$9: LED1.A, SV1.26
- new net GPI10_OUTERDOOR: PICONNECTOR.GPIO10_MOSI, R5.1
- new net GPIO11_INNERDOOR: PICONNECTOR.GPIO11_SCLK, R10.1
- new net GPIO17_J1: JP1.1, PICONNECTOR.GPIO17, R1.1
- new net GPIO22_J2: JP2.1, PICONNECTOR.GPIO22, R2.1
- net +12V: now also D1.C
- net +3V3: now also PICONNECTOR.3V3@1; no longer SV1.1
- net GND: now also C3.-, PICONNECTOR.GND@25, PICONNECTOR.GND@9; no longer SV1.25
- net N$13: now also LED1.A, PICONNECTOR.GPIO7,SPI0_CE1; no longer Q1.D, SV2.1
- net N$2: now also D1.A, Q1.D, SV2.1; no longer R10.1, SV1.18
- net VCC: now also C3.+, PICONNECTOR.5V@2, PICONNECTOR.5V@4; no longer SV1.2
Other:
- note added: "Inner door"
- note added: "Outer door"
- moved on the sheet: C1, C2, IC2, LED1, R1
